File: power.sch (KiCad schematic (older format))
At the start: 27 parts, among them J101 5V INPUT, SW101 POWER, U101 MC34063EBN, U102 LM7905_TO220

Commit message: Correct Mouser part number for R103. Was 2K, should be 22K.
Parts:
- R103: Mouser 603-CFR-25JR-522K -> 603-CFR-25JR-5222K
Changed lines of the file:
@@
 F 2 "Passive:RESA500" H 6050 4000 50  0001 C CNN
 F 3 "~" H 6050 4000 50  0001 C CNN
-F 4 "603-CFR-25JR-522K" H 1000 1950 50  0001 C CNN "Mouser"
+F 4 "603-CFR-25JR-5222K" H 1000 1950 50  0001 C CNN "Mouser"
 	1    6050 4000
 	0    1    1    0
